File: pcb_honey-jar-filler/pcb_honey-jar-filler.kicad_sch (KiCad schematic)
At the start: 76 parts, among them J1 12V, 5V, J10 OLED_3v3, GND, J11 OLED_SDA, SCL, J12 MOS out (COM, Drain), J13 230V Heater, J14 3V3, J15 12V, 5V, J16 LED2, J17 GND, J18 GND, J19 Servo, J2 12V, J20 Conn_01x07_Pin, J21 LED1, J22 Reserve, J23 Relay fallback, J24 load-cell (red, black), J25 load-cell (white, green), J26 B+ B- (free), J27 Supply, J3 3V3, J4 button1, button2, J5 4...7V, J6 Encoder A, B, J7 Encoder Button, Pos-sw, J8 MOS out (COM, Drain), J9 Motor_1 + -, K1 RT314A24, K2 RT314A24, K3 RT314A24, K4 RT314A24, K5 RT314A24, M1 DC-worm-gear motor (Carousell), Q1 IRLB8721PBF, Q2 IRLB8721PBF, U1 esp32-devkit-v1_30Pin, U10 LM2576T-ADJ, U3 ULN2003, U4 HX711_24-bit-ADC_weight-scale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, U9 LM2576T-5

Commit message: pcb: arrange parts, re-assign, add servo-cutoff
Parts:
- removed D10, D11: D, Diode_THT:D_T-1_P12.70mm_Horizontal, symbol Device:D
- removed J23: Relay fallback, terminals_libJonny:ScrewTerminal_P5mm_3Pin_FP15x8, symbol Connector:Screw_Terminal_01x03
- removed JP4, JP5, JP6, JP7: Jumper_2_Bridged, Connector_PinHeader_2.54mm:PinHeader_1x02_P2.54mm_Vertical, symbol Jumper:Jumper_2_Bridged
- removed K1, K5: RT314A24, Relay_THT:Relay_SPDT_Schrack-RT1-16A-FormC_RM5mm, symbol Relay:RT314A24
- removed M1: DC-worm-gear motor (Carousell), terminals_libJonny:ScrewTerminal_P5mm_2Pin_FP10x8, symbol Motor:Motor_DC
- added C11: 15u, Capacitor_THT:CP_Radial_D6.3mm_P2.50mm, symbol Device:C_Polarized
- added C12: 2200uF, Capacitor_THT:CP_Radial_D10.0mm_P5.00mm, symbol Device:C_Polarized
- added D12: 1N5822, Diode_THT:D_DO-201AD_P15.24mm_Horizontal, symbol Diode:1N5822
- added D13, D14: D, Diode_THT:D_T-1_P12.70mm_Horizontal, symbol Device:D
- added H1, H2, H3, H4: MountingHole, MountingHole:MountingHole_4.3mm_M4_DIN965, symbol Mechanical:MountingHole
- added J28: Relay fallback, terminals_libJonny:ScrewTerminal_P5mm_3Pin_FP15x8, symbol Connector:Screw_Terminal_01x03
- added JP10, JP11, JP12, JP9: Jumper_2_Bridged, Connector_PinHeader_2.54mm:PinHeader_1x02_P2.54mm_Vertical, symbol Jumper:Jumper_2_Bridged
- added JP8: Force-on-servo, Connector_PinHeader_2.54mm:PinHeader_1x02_P2.54mm_Vertical, symbol Jumper:Jumper_2_Bridged
- added K6, K7: Relay_LEG-xxF, relays_libJonny:Relay_LEG-xxF, symbol relays_libJonny:Relay_LEG-xxF
- added M2: DC-worm-gear motor (Carousell), terminals_libJonny:ScrewTerminal_P5mm_2Pin_FP10x8, symbol Motor:Motor_DC
- added Q6: IRF5305, Package_TO_SOT_THT:TO-220-3_Vertical, symbol Transistor_MOSFET_AKL:IRF5305
- added R18: 5k6, Resistor_THT:R_Axial_DIN0207_L6.3mm_D2.5mm_P10.16mm_Horizontal, symbol Device:R
- added R19: 2k2, Resistor_THT:R_Axial_DIN0207_L6.3mm_D2.5mm_P10.16mm_Horizontal, symbol Device:R
- added R83: 47k, Resistor_THT:R_Axial_DIN0207_L6.3mm_D2.5mm_P10.16mm_Horizontal, symbol Device:R
- added RV3: 10k, resistors_libJonny:Potentiometer_Piher_PT-10-V10_Vertical, symbol Device:R_Potentiometer_Trim
- D9, F3, J22, JP1, K4: now not fitted
- L3: value 470u -> 100u
- R10, R17, R2, R8, R9: footprint Resistor_THT:R_Axial_DIN0207_L6.3mm_D2.5mm_P2.54mm_Vertical -> Resistor_THT:R_Axial_DIN0207_L6.3mm_D2.5mm_P10.16mm_Horizontal
Connections:
- net FREE is gone; now on net OD_Relay-reserve: J20.1 (Pin_1), U3.10 (O7)
- net +12V: now also D14.1 (K), JP9.2 (B), K6.A1, K7.A1
- net +5V: now also D12.2 (A); no longer U1.15 (VIN)
- net 4...7V: now also JP8.2 (B), Q6.3 (S), R83.2, RV3.1, RV3.2; no longer J19.1 (Pin_1), U10.4 (FB)
- net GND: now also U1.14 (GND), U1.17 (GND), C11.2, C12.2, D13.2 (A), JP10.1 (A), M2.2 (-), R19.2
- net GPIO-IN_Button1: now also U1.6 (GPIO32/ADC1-CH4)
- net GPIO-IN_Button2: now also U1.7 (GPIO33/ADC1-CH5)
- net GPIO-IN_Encoder-A: now also U1.2 (GPIO36/ADC1-CH0/SENSOR_VP/[IN-ONLY])
- net GPIO-IN_Encoder-B: now also U1.3 (GPIO39/ADC1-CH3/SENSOR_VN/[IN-ONLY])
- net GPIO-IN_Encoder-Button: now also U1.4 (GPIO34/ADC1-CH6//[IN-ONLY])
- net GPIO-IN_Position-SW: now also U1.5 (GPIO35/ADC1-CH7/[IN-ONLY])
- net GPIO_Buzzer: now also U1.21 (GPIO16/UART2-RX), U3.2 (I2); no longer U3.1 (I1)
- net GPIO_LED1: now also U1.8 (GPIO25/ADC2), U3.4 (I4); no longer U3.3 (I3)
- net GPIO_LED2: now also U1.22 (GPIO17/UART2-TX), U3.3 (I3); no longer U3.2 (I2)
- net GPIO_MOS-reserve: now also U1.23 (GPIO5/VSPI-CS)
- net GPIO_MOS-valve: now also U1.24 (GPIO18/VSPI_CLK)
- net GPIO_Relay-heater: now also U1.9 (GPIO26/ADC2), U3.5 (I5); no longer U3.6 (I6)
- net GPIO_Relay-motor: now also U1.10 (GPIO27/ADC2), U3.6 (I6); no longer U3.5 (I5)
- net GPIO_Relay-reserve: now also U1.11 (GPIO14/ADC2/HSPI_CLK), U3.7 (I7); no longer U3.4 (I4)
- net HX711_DT: now also U1.12 (GPIO12/HSPI-MISO/MTDI/[LOW-AT-BOOT])
- net HX711_SCK: now also U1.13 (GPIO13/HSPI-MOSI)
- net I2C-SCL_OLED: now also U1.29 (GPIO22/I2C-SCL)
- net I2C-SDA_OLED: now also U1.26 (GPIO21/I2C-SDA)
- net OD_Buzzer: now also J20.6 (Pin_6), U3.15 (O2); no longer J20.7 (Pin_7), U3.16 (O1)
- net OD_LED1: now also J20.4 (Pin_4), U3.13 (O4); no longer J20.5 (Pin_5), U3.14 (O3)
- net OD_LED2: now also J20.5 (Pin_5), U3.14 (O3); no longer J20.6 (Pin_6), U3.15 (O2)
- net OD_Relay-heater: now also J20.3 (Pin_3), U3.12 (O5); no longer J20.2 (Pin_2), U3.11 (O6)
- net OD_Relay-motor: now also J20.2 (Pin_2), U3.11 (O6), JP12.1 (A); no longer J20.3 (Pin_3), U3.12 (O5)
- net OD_Relay-reserve: no longer J20.4 (Pin_4), U3.13 (O4)
- net Servo-PWM-Signal: now also U1.20 (GPIO4/ADC2)
- net at U1.1 (EN): now also C11.1
- net GPIO_EN-Servo-pwr: now reaches U1.19 (GPIO2/ADC2/[OnboardBlueLED+10k_down])
- net GPIO_EN-Servo-pwr: now also U3.1 (I1)
- net at F1.1: now also K6.11
- net at J13.1 (Pin_1): now also K6.12
- net at J13.2 (Pin_2): now also F1.2
- net at D22.2 (A), JP2.2 (B): now also K6.A2
- net at J13.3 (Pin_3): now also K6.14; no longer F1.2
- new net: R18.2, R19.1, U10.4 (FB)
- new net: D14.2 (A), JP12.2 (B), K7.A2
- new net: D12.1 (K), U1.15 (VIN)
- new net: D13.1 (K), JP11.1 (A), M2.1 (+)
- new net: J28.2 (Pin_2), JP11.2 (B), K7.11
- new net: J28.1 (Pin_1), JP10.2 (B), K7.12
- new net: J28.3 (Pin_3), JP9.1 (A), K7.14
- new net: C12.1, J19.1 (Pin_1), JP8.1 (A), Q6.2 (D)
- new net: R18.1, RV3.3
- new net OD_EN-Servo-pwr: J20.7 (Pin_7), Q6.1 (G), R83.1, U3.16 (O1)
- no-connect marks 0 -> 2
Other:
- note added: "12V Supply"
- note added: "1: used for USB 3: used for USB"
- note added: "Adjustable 4V...9.9V"
- note added: "Darlington Array"
- note added: "Digital Inputs"
- note added: "Load Cell"
- note added: "Mosfet outputs"
- note added: "TODO: - Servo cutoff P-MOS ? - pick regulator L"
- note added: "TODO: Pick inductor"
- note added: "Vout = 1.23 V × (1 + R1/R2)"
- note removed: "12V Supply (voltage filter)"
- note removed: "TODO: Adj circuit"
- moved on the sheet: BZ2, D22, D3, D8, F1, J1, J10, J11, J12, J13, J15, J16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

Commit message: pcb: initial routing complete, some terminals -> JST connector
Parts:
- removed H2, H3, H4: MountingHole, MountingHole:MountingHole_4.3mm_M4_DIN965, symbol Mechanical:MountingHole
- removed J10: OLED_3v3, GND, terminals_libJonny:ScrewTerminal_P3.5mm_2Pin_FP7x7, symbol Connector:Screw_Terminal_01x02
- removed J11: OLED_SDA, SCL, terminals_libJonny:ScrewTerminal_P3.5mm_2Pin_FP7x7, symbol Connector:Screw_Terminal_01x02
- removed J16: LED2, terminals_libJonny:ScrewTerminal_P3.5mm_2Pin_FP7x7, symbol Connector:Screw_Terminal_01x02
- removed J21: LED1, terminals_libJonny:ScrewTerminal_P3.5mm_2Pin_FP7x7, symbol Connector:Screw_Terminal_01x02
- removed J6: Encoder A, B, terminals_libJonny:ScrewTerminal_P3.5mm_2Pin_FP7x7, symbol Connector:Screw_Terminal_01x02
- removed J7: Encoder Button, Pos-sw, terminals_libJonny:ScrewTerminal_P3.5mm_2Pin_FP7x7, symbol Connector:Screw_Terminal_01x02
- removed JP12, JP2: Jumper_2_Bridged, Connector_PinHeader_2.54mm:PinHeader_1x02_P2.54mm_Vertical, symbol Jumper:Jumper_2_Bridged
- added H2, H3, H4, H5, H6: MountingHole_Pad, mountingHoles_libJonny:MountingHole_2.2mm_NPTH-with-pad_DRC-clearance-error, symbol Mechanical:MountingHole_Pad
- added J23, J29, J6: Conn_01x02_Pin, Connector_JST:JST_XH_B2B-XH-A_1x02_P2.50mm_Vertical, symbol Connector:Conn_01x02_Pin
- added J30: Conn_01x04_Pin, Connector_JST:JST_XH_B4B-XH-A_1x04_P2.50mm_Vertical, symbol Connector:Conn_01x04_Pin
- added J31: Conn_01x05_Pin, Connector_JST:JST_XH_B5B-XH-A_1x05_P2.50mm_Vertical, symbol Connector:Conn_01x05_Pin
- added J7: Conn_01x06_Pin, Connector_JST:JST_XH_B6B-XH-A_1x06_P2.50mm_Vertical, symbol Connector:Conn_01x06_Pin
- D13, D14: footprint Diode_THT:D_T-1_P12.70mm_Horizontal -> Diode_THT:D_T-1_P2.54mm_Vertical_KathodeUp
- F1: footprint misc_libJonny:Fuseholder_Automotive-Mini_Fuse11x4x16_Footprint15x5_Inline -> Fuse:Fuseholder_Cylinder-5x20mm_Stelvio-Kontek_PTF78_Horizontal_Open
- H1: footprint MountingHole:MountingHole_4.3mm_M4_DIN965 -> MountingHole:MountingHole_3mm
- J1: value 12V, 5V -> 12V
- J15: value 12V, 5V -> 5V
- J24, J25, JP3: now not fitted
- J4: value button1, button2 -> reserve Buttons
- L2: value 330u -> 100u; footprint Inductor_THT:L_Radial_D10.5mm_P5.00mm_Abacron_AISR-01 -> Inductor_THT:L_Toroid_Vertical_L14.0mm_W6.3mm_P4.57mm_Pulse_A
- L3: footprint Inductor_THT:L_Toroid_Vertical_L21.6mm_W11.4mm_P7.62mm_Pulse_KM-3 -> Inductor_THT:L_Toroid_Vertical_L14.0mm_W6.3mm_P4.57mm_Pulse_A
Connections:
- net +24V filtered is gone; now on net +12V: C5.1, C7.1, U10.1 (VIN), U9.1 (VIN)
- net +12V: now also J1.1 (Pin_1); no longer J15.2 (Pin_2)
- net +3V3: now also J30.4 (Pin_4), J31.5 (Pin_5)
- net +5V: now also J15.2 (Pin_2); no longer J1.1 (Pin_1)
- net GND: now also H2.1, H3.1, H4.1, H5.1, H6.1, J30.1 (Pin_1), J31.1 (Pin_1), J6.2 (Pin_2)
- net GPIO_Buzzer: now also U1.22 (GPIO17/UART2-TX), U3.3 (I3); no longer U1.21 (GPIO16/UART2-RX), U3.2 (I2)
- net GPIO_EN-Servo-pwr: now also U1.21 (GPIO16/UART2-RX), U3.2 (I2); no longer U1.19 (GPIO2/ADC2/[OnboardBlueLED+10k_down]), U3.1 (I1)
- net GPIO_LED1: now also U1.9 (GPIO26/ADC2), U3.5 (I5); no longer U1.8 (GPIO25/ADC2), U3.4 (I4)
- net GPIO_LED2: now also U1.8 (GPIO25/ADC2), U3.4 (I4); no longer U1.22 (GPIO17/UART2-TX), U3.3 (I3)
- net GPIO_MOS-reserve: now also U1.24 (GPIO18/VSPI_CLK); no longer U1.23 (GPIO5/VSPI-CS)
- net GPIO_MOS-valve: now also U1.23 (GPIO5/VSPI-CS); no longer U1.24 (GPIO18/VSPI_CLK)
- net GPIO_Relay-heater: now also U1.19 (GPIO2/ADC2/[OnboardBlueLED+10k_down]), U3.1 (I1); no longer U1.9 (GPIO26/ADC2), U3.5 (I5)
- net I2C-SCL_OLED: now also J30.2 (Pin_2)
- net I2C-SDA_OLED: now also J30.3 (Pin_3)
- net OD_Buzzer: now also J20.5 (Pin_5), U3.14 (O3); no longer J20.6 (Pin_6), U3.15 (O2)
- net OD_EN-Servo-pwr: now also J20.6 (Pin_6), U3.15 (O2); no longer J20.7 (Pin_7), U3.16 (O1)
- net OD_LED1: now also J20.3 (Pin_3), U3.12 (O5), J23.1 (Pin_1); no longer J20.4 (Pin_4), U3.13 (O4)
- net OD_LED2: now also J20.4 (Pin_4), U3.13 (O4), J29.1 (Pin_1); no longer J20.5 (Pin_5), U3.14 (O3)
- net OD_Relay-heater: now also D22.2 (A), J20.7 (Pin_7), K6.A2, U3.16 (O1); no longer J20.3 (Pin_3), U3.12 (O5)
- net OD_Relay-motor: now also D14.2 (A), K7.A2
- net at J24.2 (Pin_2), U4.1 (E+): now also J7.1 (Pin_1)
- net at J24.1 (Pin_1), U4.2 (E-): now also J7.2 (Pin_2)
- net at J25.1 (Pin_1), U4.3 (A-): now also J7.3 (Pin_3)
- net at J25.2 (Pin_2), U4.4 (A+): now also J7.4 (Pin_4)
- net at J26.1 (Pin_1), U4.5 (B-): now also J7.5 (Pin_5)
- net at J26.2 (Pin_2), U4.6 (B+): now also J7.6 (Pin_6)
- net at R17.2: now also J23.2 (Pin_2)
- net at JP11.2 (B), K7.11: now also J28.3 (Pin_3); no longer J28.2 (Pin_2)
- net at F1.2: now also J13.3 (Pin_3); no longer J13.2 (Pin_2)
- net at JP10.2 (B), K7.12: now also J28.2 (Pin_2); no longer J28.1 (Pin_1)
- net at JP9.1 (A), K7.14: now also J28.1 (Pin_1); no longer J28.3 (Pin_3)
- net at R10.2: now also J29.2 (Pin_2)
- net at J13.1 (Pin_1): now also K6.14; no longer K6.12
- new net: J13.2 (Pin_2), K6.12
- new net Encoder-A: J31.4 (Pin_4)
- new net Encoder-B: J31.3 (Pin_3)
- new net Encoder-btn: J31.2 (Pin_2)
- new net Pos-SW: J6.1 (Pin_1)
Other:
- note removed: "330uH picked for ~1A max out current"
- moved on the sheet: J1, J13, J15, J28

Commit message: pcb: Add text, testpoints, i2c-pull, Cleanup - DRC-pass
Parts:
- added J10: GPIO19, Connector_PinHeader_2.54mm:PinHeader_1x01_P2.54mm_Vertical, symbol Connector:Conn_01x01_Pin
- added J11: GPIO23, Connector_PinHeader_2.54mm:PinHeader_1x01_P2.54mm_Vertical, symbol Connector:Conn_01x01_Pin
- added J16: GPIO15, Connector_PinHeader_2.54mm:PinHeader_1x01_P2.54mm_Vertical, symbol Connector:Conn_01x01_Pin
- added R20: 4k7, Resistor_THT:R_Axial_DIN0204_L3.6mm_D1.6mm_P2.54mm_Vertical, symbol Device:R
- added R21: 4k7, Resistor_THT:R_Axial_DIN0207_L6.3mm_D2.5mm_P10.16mm_Horizontal, symbol Device:R
- added TP1: GND, Connector_PinHeader_2.54mm:PinHeader_1x01_P2.54mm_Vertical, symbol Connector:TestPoint
- added TP2: 12V, Connector_PinHeader_2.54mm:PinHeader_1x01_P2.54mm_Vertical, symbol Connector:TestPoint
- added TP3: 5V, Connector_PinHeader_2.54mm:PinHeader_1x01_P2.54mm_Vertical, symbol Connector:TestPoint
- added TP4: 4-7V, Connector_PinHeader_2.54mm:PinHeader_1x01_P2.54mm_Vertical, symbol Connector:TestPoint
- added TP5: 3V3, Connector_PinHeader_2.54mm:PinHeader_1x01_P2.54mm_Vertical, symbol Connector:TestPoint
- added TP7: SDA, Connector_PinHeader_2.54mm:PinHeader_1x01_P2.54mm_Vertical, symbol Connector:TestPoint
- added TP8: SCL, Connector_PinHeader_2.54mm:PinHeader_1x01_P2.54mm_Vertical, symbol Connector:TestPoint
- J12: value MOS out (COM, Drain) -> MOS2 out (COM, Drain)
- J14: value 3V3 -> 5V
- J23: value Conn_01x02_Pin -> LED1
- J29: value Conn_01x02_Pin -> LED2
- J30: value Conn_01x04_Pin -> OLED
- J31: value Conn_01x05_Pin -> rotary-encoder
- J6: value Conn_01x02_Pin -> Pos-switch
- J7: value Conn_01x06_Pin -> Bridge (HX711 input)
- J8: value MOS out (COM, Drain) -> MOS1 out (COM, Drain)
- TP6: value BATT -> supply; footprint Connector_PinHeader_1.00mm:PinHeader_1x01_P1.00mm_Vertical -> Connector_PinHeader_2.54mm:PinHeader_1x01_P2.54mm_Vertical; now not fitted; now left out of the parts list
Connections:
- net +12V: now also TP2.1; no longer TP6.1
- net +3V3: now also R20.1, R21.2, TP5.1
- net +5V: now also TP3.1
- net 12V-supply: now also TP6.1
- net 4...7V: now also TP4.1
- net GND: now also TP1.1
- net I2C-SCL_OLED: now also R21.1, TP8.1
- net I2C-SDA_OLED: now also R20.2, TP7.1
- net OD_Relay-reserve: no longer J20.1 (Pin_1), U3.10 (O7)
- net at U1.18 (GPIO15/HSPI_CS/MTDO/[HIGH-AT-BOOT]): now also J16.1 (Pin_1)
- net at U1.25 (GPIO19/VSPI-MISO): now also J10.1 (Pin_1)
- net at U1.30 (GPIO23/VSPI-MOSI): now also J11.1 (Pin_1)
- net GPIO_Relay-reserve renamed GPIO_OD-reserve
- new net OD_FREE: J20.1 (Pin_1), U3.10 (O7)
Other:
- note added: "Breakout board regulator supplies 3V3 to pcb"
- note added: "FREE Pins"
- note added: "Mounting holes"
- note added: "Open-Drain outputs"
- note added: "Power terminals, testpoints"
- note added: "Prevent USB backfeeding into board"
- note removed: "Power terminals"
- note removed: "TODO: - Servo cutoff P-MOS ? - pick regulator L"
- moved on the sheet: BZ2, C12, C5, C6, C7, C8, D12, D3, D4, D5, D8, D9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

Commit message: pcb: Add MOS pulldowns, Schematic cleanup
Parts:
- removed D2, D6, D7: D, Diode_THT:D_T-1_P12.70mm_Horizontal, symbol Device:D
- removed J9: Motor_1 + -, terminals_libJonny:ScrewTerminal_P5mm_2Pin_FP10x8, symbol Connector:Screw_Terminal_01x02
- removed K2, K3: RT314A24, Relay_THT:Relay_SPDT_Schrack-RT1-16A-FormC_RM5mm, symbol Relay:RT314A24
- added R22, R23: 47k, Resistor_THT:R_Axial_DIN0207_L6.3mm_D2.5mm_P10.16mm_Horizontal, symbol Device:R
- J12: value MOS2 out (COM, Drain) -> MOS2 out (FWD, Drain)
- J7: value Bridge (HX711 input) -> Load-cell (HX711 input)
- J8: value MOS1 out (COM, Drain) -> MOS1 out (FWD, Drain)
- JP10, JP11, JP9: value Jumper_2_Bridged -> EN_motor
- R10: value 330 -> 220
Connections:
- net GND: now also R22.1, R23.1
- net at Q1.1 (G), R8.2: now also R22.2
- net at Q2.1 (G), R9.2: now also R23.2
Other:
- note added: "1x Relay 230V (Heater, Reserve) 1x Relay DC / Motor-control (drive, brake)"
- note added: "All jumpers closed: - relay on: Motor ON (12V, GND) - relay off: Motor braking (GND, GND) All jumpers open: - fallback, use relay normally with 3-pin-screw terminal (NO, NC, COM)"
- note added: "P-Channel MOS"
- note removed: "24V Motor ~3A medium load"
- note removed: "2x Relay (Heater, Reserve) 1x Relay Motor (drive, brake)"
- note removed: "TODO: Pick inductor"
- title: (none) -> honey jar filler control
- moved on the sheet: C11, D22, D8, D9, F1, F3, J1, J12, J13, J15, J22, J24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

Commit message: pcb: Arrange fab text, Annotate for soldering, Fix "PWM" text
Parts:
- K6, K7: value Relay_LEG-xxF -> Relay_LEG-12
Changed lines of the file:
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@@
 			)
 		)
-		(property "Value" "Relay_LEG-xxF"
+		(property "Value" "Relay_LEG-12"
 			(at 274.32 37.846 0)
 			(effects
@@
 			)
 		)
-		(property "Value" "Relay_LEG-xxF"
+		(property "Value" "Relay_LEG-12"
 			(at 359.41 38.1 0)
 			(effects
