File: pcb_honey-jar-filler/pcb_honey-jar-filler.kicad_sch (KiCad schematic)
At the start: 97 parts, among them J1 12V, J10 GPIO19, J11 GPIO23, J12 MOS2 out (FWD, Drain), J13 230V Heater, J14 5V, J15 5V, J16 GPIO15, J17 GND, J18 GND, J19 Servo, J2 12V, J20 Conn_01x07_Pin, J22 Reserve, J23 LED1, J24 load-cell (red, black), J25 load-cell (white, green), J26 B+ B- (free), J27 Supply, J28 Relay fallback, J29 LED2, J3 3V3, J30 OLED, J31 rotary-encoder, J4 reserve Buttons, J5 4...7V, J6 Pos-switch, J7 Load-cell (HX711 input), J8 MOS1 out (FWD, Drain), K4 RT314A24, K6 Relay_LEG-12, K7 Relay_LEG-12, M2 DC-worm-gear motor (Carousell), Q1 IRLB8721PBF, Q2 IRLB8721PBF, Q6 IRF5305, U1 esp32-devkit-v1_30Pin, U10 LM2576T-ADJ, U3 ULN2003, U4 HX711_24-bit-ADC_weight-scale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, U9 LM2576T-5

Commit message: PCB: Optimize Schematic layout for thesis exports (Servo supply + Motor relay)
Parts:
- removed D9: D, Diode_THT:D_T-1_P12.70mm_Horizontal, symbol Device:D
- removed F3: F-Heater, misc_libJonny:Fuseholder_Automotive-Mini_Fuse11x4x16_Footprint15x5_Inline, symbol Device:Fuse
- removed J22: Reserve, terminals_libJonny:ScrewTerminal_P5mm_3Pin_FP15x8, symbol Connector:Screw_Terminal_01x03
- removed JP1: Jumper_2_Bridged, Connector_PinHeader_2.54mm:PinHeader_1x02_P2.54mm_Vertical, symbol Jumper:Jumper_2_Bridged
- removed K4: RT314A24, Relay_THT:Relay_SPDT_Schrack-RT1-16A-FormC_RM5mm, symbol Relay:RT314A24
- D13: value D -> 1N5822
- J28: value Relay fallback -> Relay (non-motor mode)
- J5: value 4...7V -> 4...10V
- M2: value DC-worm-gear motor (Carousell) -> DC-worm-gear motor (Carousel)
- renumbered RV3 to R1.1, R18 to R1.2, R19 to R2
Connections:
- net feedback: now reaches R1.2.2, R2.1, U10.4 (FB)
- net 4...7V renamed 4...10V
Other:
- note added: "Adjustable 4V...9.95V"
- note added: "Adjustable Servo Power Supply 4.4-10 V (Buck Converter)"
- note added: "All jumpers closed: - relay on: Motor driven (12V, GND) - relay off: Motor braking (GND, GND) All jumpers open: - non-motor mode, use relay normally with 3-pin-screw terminal (NO, NC, COM)"
- note added: "Relay 230V (Heater, Reserve)"
- note added: "Relay for motor drive (drive, brake)"
- note added: "max 3 A"
- note removed: "1x Relay 230V (Heater, Reserve) 1x Relay DC / Motor-control (drive, brake)"
- note removed: "4..7V Supply Servo (buck converter)"
- note removed: "470uH picked for ~1.3A max out current"
- note removed: "Adjustable 4V...9.9V"
- note removed: "All jumpers closed: - relay on: Motor ON (12V, GND) - relay off: Motor braking (GND, GND) All jumpers open: - fallback, use relay normally with 3-pin-screw terminal (NO, NC, COM)"
- moved on the sheet: C7, C8, D13, D14, D22, D3, D5, D8, F1, J1, J12, J13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
