File: pcb_honey-jar-filler/pcb_honey-jar-filler_THESIS.kicad_sch (KiCad schematic)
At the start: 92 parts, among them J1 12V, J10 GPIO19, J11 GPIO23, J12 MOS2 out (FWD, Drain), J13 230V Heater, J14 5V, J15 5V, J16 GPIO15, J17 GND, J18 GND, J19 Servo, J2 12V, J20 Conn_01x07_Pin, J23 LED1, J24 load-cell (red, black), J25 load-cell (white, green), J26 B+ B- (free), J27 Supply, J28 Relay (non-motor mode), J29 LED2, J3 3V3, J30 OLED, J31 rotary-encoder, J4 reserve Buttons, J5 4...10V, J6 Pos-switch, J7 Load-cell (HX711 input), J8 MOS1 out (FWD, Drain), K6 Relay_LEG-12, K7 Relay_LEG-12, M2 DC-worm-gear motor (Carousel), Q1 IRLB8721PBF, Q2 IRLB8721PBF, Q6 IRF5305, U1 esp32-devkit-v1_30Pin, U10 LM2576T-ADJ, U3 ULN2003, U4 HX711_24-bit-ADC_weight-scale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, U9 LM2576T-5

Commit message: PCB: Optimize schematic layout, Add thesis schematic version
Parts:
- added C13: \${C_filter}, capacitor_libJonny:C_DualType__Disc-7.0x2.5mm-P5mm__Elko-D5mm-P2.5mm, symbol Device:C
- added R18: \${R_pullup}, Resistor_THT:R_Axial_DIN0207_L6.3mm_D2.5mm_P10.16mm_Horizontal, symbol Device:R
- added R19: \${R_series}, Resistor_THT:R_Axial_DIN0207_L6.3mm_D2.5mm_P10.16mm_Horizontal, symbol Device:R
Connections:
- net +3V3: now also R18.1; no longer U1.16 (3V3)
- net +5V: no longer D12.2 (A)
- net GND: now also C13.2
- new net GPIO: C13.1, R19.2
- new net switch-terminal: R18.2, R19.1
Other:
- note added: "1/1"
- note added: "Digital- Input-Filter"
- note added: "Relay for 12V motor (drive, brake)"
- note added: "external switch pulls this to GND when actuated"
- note added: "microcontroller"
- note removed: "HX711_DT currently wired to GPIO19"
- note removed: "Relay for motor drive (drive, brake)"
- note removed: "TODO next version: - Critical: do not use GPIO12 for HX711_DT (strapping pin) -> reroute - Add connector for front button input (currently using reserve terminal) - Add connector + decoupling for RGB LED-Strip - optimize servo power (optional, works currently) - Add additional decoupling C for servo power - Switch to 5A regulator"
- moved on the sheet: BZ2, C11, C12, D12, D8, J1, J10, J11, J12, J15, J16, J23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
